Commit message: Fix urdf mesh paths

File: urdf/sick_lms1xx.urdf.xacro (robot description, xacro)
@@ -13,5 +13,5 @@
       <visual>
         <geometry>
-          <mesh filename="package://sick_scan/meshes/LMS1xx_small.dae" />
+          <mesh filename="package://sick_scan_xd/meshes/LMS1xx_small.dae" />
         </geometry>
         <material name="blue" >
@@ -21,5 +21,5 @@
       <collision>
         <geometry>
-          <mesh filename="package://sick_scan/meshes/LMS1xx_collision.stl" />
+          <mesh filename="package://sick_scan_xd/meshes/LMS1xx_collision.stl" />
         </geometry>
       </collision>

File: urdf/sick_lms5xx.urdf.xacro (robot description, xacro)
@@ -13,5 +13,5 @@
       <visual>
         <geometry>
-          <mesh filename="package://sick_scan/meshes/LMS5xx_small.dae" />
+          <mesh filename="package://sick_scan_xd/meshes/LMS5xx_small.dae" />
         </geometry>
         <material name="blue" >
@@ -21,5 +21,5 @@
       <collision>
         <geometry>
-          <mesh filename="package://sick_scan/meshes/LMS5xx_collision.stl" />
+          <mesh filename="package://sick_scan_xd/meshes/LMS5xx_collision.stl" />
         </geometry>
       </collision>

File: urdf/sick_scan.urdf.xacro (robot description, xacro)
@@ -9,5 +9,5 @@
       min_angle="${min_angle}" max_angle="${max_angle}"
       min_range="0.05" max_range="4.0" gaussian_noise="${gaussian_noise}" samples="${samples}"
-      mesh="package://sick_scan/meshes/sick_tim_5xx.stl" />
+      mesh="package://sick_scan_xd/meshes/sick_tim_5xx.stl" />
   </xacro:macro>
   <xacro:macro name="sick_tim_56x" params="name ros_topic min_angle:=-2.357 max_angle:=2.357 gaussian_noise:=0.01 samples:=811">
@@ -16,5 +16,5 @@
       min_angle="${min_angle}" max_angle="${max_angle}"
       min_range="0.05" max_range="10.0" gaussian_noise="${gaussian_noise}" samples="${samples}"
-      mesh="package://sick_scan/meshes/sick_tim_5xx.stl" />
+      mesh="package://sick_scan_xd/meshes/sick_tim_5xx.stl" />
   </xacro:macro>
   <xacro:macro name="sick_tim_57x" params="name ros_topic min_angle:=-2.357 max_angle:=2.357 gaussian_noise:=0.01 samples:=811">
@@ -23,5 +23,5 @@
       min_angle="${min_angle}" max_angle="${max_angle}"
       min_range="0.05" max_range="25.0" gaussian_noise="${gaussian_noise}" samples="${samples}"
-      mesh="package://sick_scan/meshes/sick_tim_5xx.stl" />
+      mesh="package://sick_scan_xd/meshes/sick_tim_5xx.stl" />
   </xacro:macro>
   <xacro:macro name="sick_tim_1xxx" params="name ros_topic min_angle:=-2.357 max_angle:=2.357 gaussian_noise:=0.015 samples:=271">
@@ -30,5 +30,5 @@
       min_angle="${min_angle}" max_angle="${max_angle}"
       min_range="0.05" max_range="4.0" gaussian_noise="${gaussian_noise}" samples="${samples}"
-      mesh="package://sick_scan/meshes/sick_tim_1xxx.stl" />
+      mesh="package://sick_scan_xd/meshes/sick_tim_1xxx.stl" />
   </xacro:macro>
   <xacro:macro name="sick_tim" params="name ros_topic length width height mass z_offset min_angle max_angle min_range max_range gaussian_noise samples mesh">
